File: HW/BSidesPDX_2018/BSidesPDX_2018.sch (KiCad schematic (older format))
At the start: 3 parts

Commit message: added SAO connector to local library. Added 5 SAO to schematic
Parts:
- removed BT1: Battery, symbol Device:Battery
- removed D1: LED, symbol Device:LED
- added X? (x5): Badgelife_shitty_connector, symbol BSidesPDX_2018:Badgelife_shitty_connector
Connections:
- wire segments 7 -> 0
Changed lines of the file:
@@
 $EndDescr
-$Comp
-L Device:LED D1
-U 1 1 5B8A3203
-P 4460 2970
-F 0 "D1" V 4498 2853 50  0000 R CNN
-F 1 "LED" V 4407 2853 50  0000 R CNN
-F 2 "" H 4460 2970 50  0001 C CNN
-F 3 "~" H 4460 2970 50  0001 C CNN
-	1    4460 2970
-	0    -1   -1   0
-$EndComp
-$Comp
-L Device:Battery BT1
-U 1 1 5B8A336A
-P 3610 2980
-F 0 "BT1" H 3718 3026 50  0000 L CNN
-F 1 "Battery" H 3718 2935 50  0000 L CNN
-F 2 "" V 3610 3040 50  0001 C CNN
-F 3 "~" V 3610 3040 50  0001 C CNN
-	1    3610 2980
-	1    0    0    -1
-$EndComp
-Wire Wire Line
-	3610 2780 3610 2740
-Wire Wire Line
-	3610 2740 3990 2740
-Wire Wire Line
-	4290 2740 4460 2740
-Wire Wire Line
-	4460 2740 4460 2820
-Wire Wire Line
-	4460 3120 4460 3250
-Wire Wire Line
-	4460 3250 3610 3250
-Wire Wire Line
-	3610 3250 3610 3180
 $Comp
 L BSidesPDX_2018:RGB_LED D?
@@
 	1    0    0    -1
 $EndComp
+$Comp
+L BSidesPDX_2018:Badgelife_shitty_connector X?
+U 1 1 5B8DDFA4
+P 2320 5270
+F 0 "X?" H 2420 5707 60  0000 C CNN
+F 1 "Badgelife_shitty_connector" H 2420 5601 60  0000 C CNN
+F 2 "" H 2320 5270 60  0001 C CNN
+F 3 "" H 2320 5270 60  0001 C CNN
+	1    2320 5270
+	1    0    0    -1
+$EndComp
+$Comp
+L BSidesPDX_2018:Badgelife_shitty_connector X?
+U 1 1 5B8DE078
+P 3810 5290
+F 0 "X?" H 3910 5727 60  0000 C CNN
+F 1 "Badgelife_shitty_connector" H 3910 5621 60  0000 C CNN
+F 2 "" H 3810 5290 60  0001 C CNN
+F 3 "" H 3810 5290 60  0001 C CNN
+	1    3810 5290
+	1    0    0    -1
+$EndComp
+$Comp
+L BSidesPDX_2018:Badgelife_shitty_connector X?
+U 1 1 5B8DE096
+P 5200 5280
+F 0 "X?" H 5300 5717 60  0000 C CNN
+F 1 "Badgelife_shitty_connector" H 5300 5611 60  0000 C CNN
+F 2 "" H 5200 5280 60  0001 C CNN
+F 3 "" H 5200 5280 60  0001 C CNN
+	1    5200 5280
+	1    0    0    -1
+$EndComp
+$Comp
+L BSidesPDX_2018:Badgelife_shitty_connector X?
+U 1 1 5B8DE12E
+P 6640 5260
+F 0 "X?" H 6740 5697 60  0000 C CNN
+F 1 "Badgelife_shitty_connector" H 6740 5591 60  0000 C CNN
+F 2 "" H 6640 5260 60  0001 C CNN
+F 3 "" H 6640 5260 60  0001 C CNN
+	1    6640 5260
+	1    0    0    -1
+$EndComp
+$Comp
+L BSidesPDX_2018:Badgelife_shitty_connector X?
+U 1 1 5B8DE176
+P 7980 5240
+F 0 "X?" H 8080 5677 60  0000 C CNN
+F 1 "Badgelife_shitty_connector" H 8080 5571 60  0000 C CNN
+F 2 "" H 7980 5240 60  0001 C CNN
+F 3 "" H 7980 5240 60  0001 C CNN
+	1    7980 5240
+	1    0    0    -1
+$EndComp

Commit message: added SAO connectors, wires, and labels
Parts:
- removed X? (x4): Badgelife_shitty_connector, symbol BSidesPDX_2018:Badgelife_shitty_connector
- added BT?: Battery_Cell, symbol Device:Battery_Cell
- added D? (x4): LED, symbol Device:LED
- added R? (x2): R, symbol Device:R
- added X? (x4): Badgelife_shitty_connector, symbol BSidesPDX_2018:Badgelife_shitty_connector
Connections:
- net labels added: 3V0, GND, SCL, SDA
- wire segments 0 -> 43

Commit message: Added PWM busses and RGB LEDs
Parts:
- removed D?: LED, symbol Device:LED
- added D? (x3): RGB_LED, symbol BSidesPDX_2018:RGB_LED
- added R? (x3): R, symbol Device:R
Connections:
- net labels added: B_PWM, G_PWM, R_PWM
- wire segments 43 -> 87
Changed lines of the file:
@@
 $EndDescr
-$Comp
-L BSidesPDX_2018:RGB_LED D?
-U 1 1 5B8B9026
-P 5850 3550
-F 0 "D?" H 5850 3875 50  0000 C CNN
-F 1 "RGB_LED" H 5850 3784 50  0000 C CNN
-F 2 "" H 5925 3325 50  0001 C CNN
-F 3 "" H 5925 3325 50  0001 C CNN
-	1    5850 3550
-	0    1    1    0
-$EndComp
 $Comp
 L BSidesPDX_2018:Badgelife_shitty_connector X?
@@
 $EndComp
 $Comp
-L Device:LED D?
-U 1 1 5B8DEB55
-P 2640 3410
-F 0 "D?" H 2631 3626 50  0000 C CNN
-F 1 "LED" H 2631 3535 50  0000 C CNN
-F 2 "" H 2640 3410 50  0001 C CNN
-F 3 "~" H 2640 3410 50  0001 C CNN
-	1    2640 3410
-	1    0    0    -1
-$EndComp
-$Comp
 L Device:R R?
 U 1 1 5B8DEDCF
-P 5840 2950
-F 0 "R?" H 5910 2996 50  0000 L CNN
-F 1 "R" H 5910 2905 50  0000 L CNN
-F 2 "" V 5770 2950 50  0001 C CNN
-F 3 "~" H 5840 2950 50  0001 C CNN
-	1    5840 2950
+P 5710 2730
+F 0 "R?" H 5780 2776 50  0000 L CNN
+F 1 "R" H 5780 2685 50  0000 L CNN
+F 2 "" V 5640 2730 50  0001 C CNN
+F 3 "~" H 5710 2730 50  0001 C CNN
+	1    5710 2730
 	1    0    0    -1
 $EndComp
@@
 Text Label 9670 5560 0    50   ~ 0
 SCL
+Wire Wire Line
+	5710 2975 5710 2880
+Wire Wire Line
+	5710 2980 5710 2975
+Connection ~ 5710 2975
+$Comp
+L BSidesPDX_2018:RGB_LED D?
+U 1 1 5B8B9026
+P 5710 3300
+F 0 "D?" H 5710 3625 50  0000 C CNN
+F 1 "RGB_LED" H 5710 3534 50  0000 C CNN
+F 2 "" H 5785 3075 50  0001 C CNN
+F 3 "" H 5785 3075 50  0001 C CNN
+	1    5710 3300
+	0    1    1    0
+$EndComp
+Wire Wire Line
+	5710 3620 5710 3625
+Connection ~ 5710 3625
+Wire Wire Line
+	5810 3620 5810 3625
+Connection ~ 5810 3625
+Wire Wire Line
+	5610 3620 5610 3625
+Connection ~ 5610 3625
+Wire Wire Line
+	5610 3625 5610 3760
+$Comp
+L Device:R R?
+U 1 1 5B8EB873
+P 6380 2730
+F 0 "R?" H 6450 2776 50  0000 L CNN
+F 1 "R" H 6450 2685 50  0000 L CNN
+F 2 "" V 6310 2730 50  0001 C CNN
+F 3 "~" H 6380 2730 50  0001 C CNN
+	1    6380 2730
+	1    0    0    -1
+$EndComp
+Wire Wire Line
+	6380 2975 6380 2880
+Wire Wire Line
+	6380 2980 6380 2975
+Connection ~ 6380 2975
+$Comp
+L BSidesPDX_2018:RGB_LED D?
+U 1 1 5B8EB87C
+P 6380 3300
+F 0 "D?" H 6380 3625 50  0000 C CNN
+F 1 "RGB_LED" H 6380 3534 50  0000 C CNN
+F 2 "" H 6455 3075 50  0001 C CNN
+F 3 "" H 6455 3075 50  0001 C CNN
+	1    6380 3300
+	0    1    1    0
+$EndComp
+Wire Wire Line
+	6380 3620 6380 3625
+Connection ~ 6380 3625
+Wire Wire Line
+	6480 3620 6480 3625
+Connection ~ 6480 3625
+Wire Wire Line
+	6280 3620 6280 3625
+Connection ~ 6280 3625
+Wire Wire Line
+	6280 3625 6280 3760
+Wire Wire Line
+	5610 3760 6280 3760
+Wire Wire Line
+	5710 3890 6380 3890
+Wire Wire Line
+	5710 3625 5710 3890
+Wire Wire Line
+	6380 3625 6380 3890
+Wire Wire Line
+	5810 3990 6480 3990
+Wire Wire Line
+	5810 3625 5810 3990
+Wire Wire Line
+	6480 3625 6480 3990
+$Comp
+L Device:R R?
+U 1 1 5B8F20F4
+P 7000 2730
+F 0 "R?" H 7070 2776 50  0000 L CNN
+F 1 "R" H 7070 2685 50  0000 L CNN
+F 2 "" V 6930 2730 50  0001 C CNN
+F 3 "~" H 7000 2730 50  0001 C CNN
+	1    7000 2730
+	1    0    0    -1
+$EndComp
+Wire Wire Line
+	7000 2975 7000 2880
+Wire Wire Line
+	7000 2980 7000 2975
+Connection ~ 7000 2975
+$Comp
+L BSidesPDX_2018:RGB_LED D?
+U 1 1 5B8F20FD
+P 7000 3300
+F 0 "D?" H 7000 3625 50  0000 C CNN
+F 1 "RGB_LED" H 7000 3534 50  0000 C CNN
+F 2 "" H 7075 3075 50  0001 C CNN
+F 3 "" H 7075 3075 50  0001 C CNN
+	1    7000 3300
+	0    1    1    0
+$EndComp
+Wire Wire Line
+	7000 3620 7000 3625
+Connection ~ 7000 3625
+Wire Wire Line
+	7100 3620 7100 3625
+Connection ~ 7100 3625
+Wire Wire Line
+	6900 3620 6900 3625
+Connection ~ 6900 3625
+Wire Wire Line
+	6900 3625 6900 3760
+$Comp
+L Device:R R?
+U 1 1 5B8F210A
+P 7670 2730
+F 0 "R?" H 7740 2776 50  0000 L CNN
+F 1 "R" H 7740 2685 50  0000 L CNN
+F 2 "" V 7600 2730 50  0001 C CNN
+F 3 "~" H 7670 2730 50  0001 C CNN
+	1    7670 2730
+	1    0    0    -1
+$EndComp
+Wire Wire Line
+	7670 2975 7670 2880
+Wire Wire Line
+	7670 2980 7670 2975
+Connection ~ 7670 2975
+$Comp
+L BSidesPDX_2018:RGB_LED D?
+U 1 1 5B8F2113
+P 7670 3300
+F 0 "D?" H 7670 3625 50  0000 C CNN
+F 1 "RGB_LED" H 7670 3534 50  0000 C CNN
+F 2 "" H 7745 3075 50  0001 C CNN
+F 3 "" H 7745 3075 50  0001 C CNN
+	1    7670 3300
+	0    1    1    0
+$EndComp
+Wire Wire Line
+	7670 3620 7670 3625
+Connection ~ 7670 3625
+Wire Wire Line
+	7770 3620 7770 3625
+Connection ~ 7770 3625
+Wire Wire Line
+	7570 3620 7570 3625
+Connection ~ 7570 3625
+Wire Wire Line
+	7570 3625 7570 3760
+Wire Wire Line
+	7000 3625 7000 3890
+Wire Wire Line
+	7670 3625 7670 3890
+Wire Wire Line
+	7100 3625 7100 3990
+Wire Wire Line
+	6280 3760 6900 3760
+Connection ~ 6280 3760
+Connection ~ 6900 3760
+Wire Wire Line
+	6900 3760 7570 3760
+Wire Wire Line
+	6380 3890 7000 3890
+Connection ~ 6380 3890
+Connection ~ 7000 3890
+Wire Wire Line
+	7000 3890 7670 3890
+Wire Wire Line
+	6480 3990 7100 3990
+Wire Wire Line
+	7770 3625 7770 3990
+Connection ~ 6480 3990
+Connection ~ 7100 3990
+Wire Wire Line
+	7100 3990 7770 3990
+Wire Wire Line
+	5610 3760 5240 3760
+Connection ~ 5610 3760
+Wire Wire Line
+	5710 3890 5240 3890
+Connection ~ 5710 3890
+Wire Wire Line
+	5810 3990 5240 3990
+Connection ~ 5810 3990
+Text Label 5240 3760 2    50   ~ 0
+B_PWM
+Text Label 5240 3890 2    50   ~ 0
+G_PWM
+Text Label 5240 3990 2    50   ~ 0
+R_PWM
 $EndSCHEMATC

Commit message: Added resistor values. Added the first leg of CharliePlex LEDs
Parts:
- R? (x5): value R -> 100R
Connections:
- wire segments 87 -> 97
Changed lines of the file:
@@
 F 3 "~" H 2680 2360 50  0001 C CNN
 	1    2680 2360
-	1    0    0    -1
+	-1   0    0    1
 $EndComp
 $Comp
 L Device:LED D?
 U 1 1 5B8DEAB5
-P 2650 2720
-F 0 "D?" H 2641 2936 50  0000 C CNN
-F 1 "LED" H 2641 2845 50  0000 C CNN
-F 2 "" H 2650 2720 50  0001 C CNN
-F 3 "~" H 2650 2720 50  0001 C CNN
-	1    2650 2720
-	1    0    0    -1
+P 2680 2760
+F 0 "D?" H 2671 2976 50  0000 C CNN
+F 1 "LED" H 2671 2885 50  0000 C CNN
+F 2 "" H 2680 2760 50  0001 C CNN
+F 3 "~" H 2680 2760 50  0001 C CNN
+	1    2680 2760
+	-1   0    0    1
 $EndComp
 $Comp
 L Device:LED D?
 U 1 1 5B8DEAF5
-P 2640 3150
-F 0 "D?" H 2631 3366 50  0000 C CNN
-F 1 "LED" H 2631 3275 50  0000 C CNN
-F 2 "" H 2640 3150 50  0001 C CNN
-F 3 "~" H 2640 3150 50  0001 C CNN
-	1    2640 3150
-	1    0    0    -1
+P 2680 3160
+F 0 "D?" H 2671 3376 50  0000 C CNN
+F 1 "LED" H 2671 3285 50  0000 C CNN
+F 2 "" H 2680 3160 50  0001 C CNN
+F 3 "~" H 2680 3160 50  0001 C CNN
+	1    2680 3160
+	-1   0    0    1
 $EndComp
 $Comp
@@
 P 5710 2730
 F 0 "R?" H 5780 2776 50  0000 L CNN
-F 1 "R" H 5780 2685 50  0000 L CNN
+F 1 "100R" H 5780 2685 50  0000 L CNN
 F 2 "" V 5640 2730 50  0001 C CNN
 F 3 "~" H 5710 2730 50  0001 C CNN
@@
 P 2400 2020
 F 0 "R?" H 2470 2066 50  0000 L CNN
-F 1 "R" H 2470 1975 50  0000 L CNN
+F 1 "100R" H 2470 1975 50  0000 L CNN
 F 2 "" V 2330 2020 50  0001 C CNN
 F 3 "~" H 2400 2020 50  0001 C CNN
@@
 P 6380 2730
 F 0 "R?" H 6450 2776 50  0000 L CNN
-F 1 "R" H 6450 2685 50  0000 L CNN
+F 1 "100R" H 6450 2685 50  0000 L CNN
 F 2 "" V 6310 2730 50  0001 C CNN
 F 3 "~" H 6380 2730 50  0001 C CNN
@@
 P 7000 2730
 F 0 "R?" H 7070 2776 50  0000 L CNN
-F 1 "R" H 7070 2685 50  0000 L CNN
+F 1 "100R" H 7070 2685 50  0000 L CNN
 F 2 "" V 6930 2730 50  0001 C CNN
 F 3 "~" H 7000 2730 50  0001 C CNN
@@
 P 7670 2730
 F 0 "R?" H 7740 2776 50  0000 L CNN
-F 1 "R" H 7740 2685 50  0000 L CNN
+F 1 "100R" H 7740 2685 50  0000 L CNN
 F 2 "" V 7600 2730 50  0001 C CNN
 F 3 "~" H 7670 2730 50  0001 C CNN
@@
 Text Label 5240 3990 2    50   ~ 0
 R_PWM
+Wire Wire Line
+	2400 2170 2400 2360
+Wire Wire Line
+	2400 2360 2530 2360
+Wire Wire Line
+	2400 2360 2400 2760
+Wire Wire Line
+	2400 2760 2530 2760
+Connection ~ 2400 2360
+Wire Wire Line
+	2400 2760 2400 3160
+Wire Wire Line
+	2400 3160 2530 3160
+Connection ~ 2400 2760
+Wire Wire Line
+	2400 1870 2400 1710
+Wire Wire Line
+	2830 2360 3070 2360
+Wire Wire Line
+	2830 2760 3070 2760
+Wire Wire Line
+	2830 3160 3070 3160
 $EndSCHEMATC

Commit message: added MCU datasheet, added charlieplex LEDs, and MCU to schematic
Parts:
- added D? (x9): LED, symbol Device:LED
- added R? (x3): 100R, symbol Device:R
- added U?: ATtiny861A-SU, Package_SO:SOIC-20W_7.5x12.8mm_P1.27mm, symbol MCU_Microchip_ATtiny:ATtiny861A-SU
Connections:
- wire segments 97 -> 127

Commit message: lable RGB leds
Parts:
- U?: value ATtiny861A-SU -> ATTINY861-15XD
Connections:
- net labels added: EN_RGB1, EN_RGB2, EN_RGB3, EN_RGB4
- wire segments 127 -> 138
Other:
- moved on the sheet: U?

Commit message: fixed wires on RGB, LED, MCU and caps.
Parts:
- added C? (x2): C, symbol Device:C
Connections:
- wire segments 138 -> 121
Changed lines of the file:
@@
 $EndComp
-Wire Wire Line
-	9300 1575 9300 1485
-Connection ~ 9300 1485
-Wire Wire Line
-	9300 1485 9300 1475
 Wire Wire Line
 	980  6030 920  6030
@@
 Text Label 8680 6220 0    50   ~ 0
 SCL
-Wire Wire Line
-	5595 4165 5595 4070
-Wire Wire Line
-	5595 4170 5595 4165
-Connection ~ 5595 4165
 $Comp
 L BSidesPDX_2018:RGB_LED D?
@@
 	0    1    1    0
 $EndComp
-Wire Wire Line
-	5595 4810 5595 4815
-Connection ~ 5595 4815
-Wire Wire Line
-	5695 4810 5695 4815
-Connection ~ 5695 4815
-Wire Wire Line
-	5495 4810 5495 4815
-Connection ~ 5495 4815
-Wire Wire Line
-	5495 4815 5495 4950
 $Comp
 L Device:R R?
@@
 	1    0    0    -1
 $EndComp
-Wire Wire Line
-	6265 4165 6265 4070
-Wire Wire Line
-	6265 4170 6265 4165
-Connection ~ 6265 4165
 $Comp
 L BSidesPDX_2018:RGB_LED D?
@@
 	0    1    1    0
 $EndComp
-Wire Wire Line
-	6265 4810 6265 4815
-Connection ~ 6265 4815
-Wire Wire Line
-	6365 4810 6365 4815
-Connection ~ 6365 4815
-Wire Wire Line
-	6165 4810 6165 4815
-Connection ~ 6165 4815
-Wire Wire Line
-	6165 4815 6165 4950
-Wire Wire Line
-	5495 4950 6165 4950
-Wire Wire Line
-	5595 5080 6265 5080
-Wire Wire Line
-	5595 4815 5595 5080
-Wire Wire Line
-	6265 4815 6265 5080
-Wire Wire Line
-	5695 5180 6365 5180
-Wire Wire Line
-	5695 4815 5695 5180
-Wire Wire Line
-	6365 4815 6365 5180
 $Comp
 L Device:R R?
@@
 	1    0    0    -1
 $EndComp
-Wire Wire Line
-	6885 4165 6885 4070
-Wire Wire Line
-	6885 4170 6885 4165
-Connection ~ 6885 4165
 $Comp
 L BSidesPDX_2018:RGB_LED D?
@@
 	0    1    1    0
 $EndComp
-Wire Wire Line
-	6885 4810 6885 4815
-Connection ~ 6885 4815
-Wire Wire Line
-	6985 4810 6985 4815
-Connection ~ 6985 4815
-Wire Wire Line
-	6785 4810 6785 4815
-Connection ~ 6785 4815
-Wire Wire Line
-	6785 4815 6785 4950
 $Comp
 L Device:R R?
@@
 	1    0    0    -1
 $EndComp
-Wire Wire Line
-	7555 4165 7555 4070
-Wire Wire Line
-	7555 4170 7555 4165
-Connection ~ 7555 4165
 $Comp
 L BSidesPDX_2018:RGB_LED D?
@@
 	0    1    1    0
 $EndComp
-Wire Wire Line
-	7555 4810 7555 4815
-Connection ~ 7555 4815
-Wire Wire Line
-	7655 4810 7655 4815
-Connection ~ 7655 4815
-Wire Wire Line
-	7455 4810 7455 4815
-Connection ~ 7455 4815
-Wire Wire Line
-	7455 4815 7455 4950
-Wire Wire Line
-	6885 4815 6885 5080
-Wire Wire Line
-	7555 4815 7555 5080
-Wire Wire Line
-	6985 4815 6985 5180
-Wire Wire Line
-	6165 4950 6785 4950
-Connection ~ 6165 4950
-Connection ~ 6785 4950
-Wire Wire Line
-	6785 4950 7455 4950
-Wire Wire Line
-	6265 5080 6885 5080
-Connection ~ 6265 5080
-Connection ~ 6885 5080
-Wire Wire Line
-	6885 5080 7555 5080
-Wire Wire Line
-	6365 5180 6985 5180
-Wire Wire Line
-	7655 4815 7655 5180
-Connection ~ 6365 5180
-Connection ~ 6985 5180
-Wire Wire Line
-	6985 5180 7655 5180
-Wire Wire Line
-	5495 4950 5125 4950
-Connection ~ 5495 4950
-Wire Wire Line
-	5595 5080 5125 5080
-Connection ~ 5595 5080
-Wire Wire Line
-	5695 5180 5125 5180
-Connection ~ 5695 5180
 Text Label 5125 4950 2    50   ~ 0
 B_PWM
@@
 Wire Wire Line
 	8130 2935 8370 2935
+Wire Wire Line
+	2060 4230 2110 4230
+Wire Wire Line
+	2110 4230 2110 4330
+Connection ~ 2110 4230
+Wire Wire Line
+	2110 4230 2160 4230
+$Comp
+L power:GND #PWR0107
+U 1 1 5B92EDF1
+P 2110 4330
+F 0 "#PWR0107" H 2110 4080 50  0001 C CNN
+F 1 "GND" H 2115 4157 50  0000 C CNN
+F 2 "" H 2110 4330 50  0001 C CNN
+F 3 "" H 2110 4330 50  0001 C CNN
+	1    2110 4330
+	1    0    0    -1
+$EndComp
+Text Label 5595 3465 3    50   ~ 0
+EN_RGB1
+Wire Wire Line
+	5595 3465 5595 3770
+Wire Wire Line
+	6265 3770 6265 3465
+Text Label 6265 3465 3    50   ~ 0
+EN_RGB2
+Wire Wire Line
+	6885 3770 6885 3470
+Text Label 6885 3470 3    50   ~ 0
+EN_RGB3
+Wire Wire Line
+	7555 3770 7555 3470
+Text Label 7555 3470 3    50   ~ 0
+EN_RGB4
+$Comp
+L Device:C C?
+U 1 1 5B951E24
+P 10090 1345
+F 0 "C?" H 10205 1391 50  0000 L CNN
+F 1 "C" H 10205 1300 50  0000 L CNN
+F 2 "" H 10128 1195 50  0001 C CNN
+F 3 "~" H 10090 1345 50  0001 C CNN
+	1    10090 1345
+	1    0    0    -1
+$EndComp
+$Comp
+L Device:C C?
+U 1 1 5B951F0C
+P 10665 1345
+F 0 "C?" H 10780 1391 50  0000 L CNN
+F 1 "C" H 10780 1300 50  0000 L CNN
+F 2 "" H 10703 1195 50  0001 C CNN
+F 3 "~" H 10665 1345 50  0001 C CNN
+	1    10665 1345
+	1    0    0    -1
+$EndComp
+Wire Wire Line
+	10090 1195 10090 1045
+Text Label 10090 1045 0    50   ~ 0
+3V0
+Wire Wire Line
+	10665 1195 10665 1045
+Text Label 10665 1045 0    50   ~ 0
+3V0
+Wire Wire Line
+	9300 1485 9300 1575
+Wire Wire Line
+	5125 4950 5495 4950
+Wire Wire Line
+	5495 4815 5495 4950
+Connection ~ 5495 4950
+Wire Wire Line
+	5125 5080 5595 5080
+Wire Wire Line
+	5595 4815 5595 5080
+Connection ~ 5595 5080
+Wire Wire Line
+	5125 5180 5695 5180
+Wire Wire Line
+	5695 4815 5695 5180
+Connection ~ 5695 5180
+Wire Wire Line
+	6165 4815 6165 4950
+Wire Wire Line
+	5495 4950 6165 4950
+Connection ~ 6165 4950
+Wire Wire Line
+	5595 5080 6265 5080
+Wire Wire Line
+	6265 4815 6265 5080
+Connection ~ 6265 5080
+Wire Wire Line
+	5695 5180 6365 5180
+Wire Wire Line
+	6365 4815 6365 5180
+Connection ~ 6365 5180
+Wire Wire Line
+	6165 4950 6785 4950
+Wire Wire Line
+	6265 5080 6885 5080
+Wire Wire Line
+	6365 5180 6985 5180
+Wire Wire Line
+	6785 4815 6785 4950
+Connection ~ 6785 4950
+Wire Wire Line
+	6785 4950 7455 4950
+Wire Wire Line
+	6885 4815 6885 5080
+Connection ~ 6885 5080
+Wire Wire Line
+	6885 5080 7555 5080
+Wire Wire Line
+	6985 4815 6985 5180
+Connection ~ 6985 5180
+Wire Wire Line
+	6985 5180 7655 5180
+Wire Wire Line
+	5595 4165 5595 4070
+Wire Wire Line
+	7455 4950 7455 4815
+Wire Wire Line
+	7555 5080 7555 4815
+Wire Wire Line
+	7655 4815 7655 5180
+Wire Wire Line
+	6265 4165 6265 4070
+Wire Wire Line
+	7555 4070 7555 4165
 $Comp
 L MCU_Microchip_ATtiny:ATtiny861A-SU U?
@@
 $EndComp
 Wire Wire Line
-	2060 4010 2060 4015
-Wire Wire Line
-	2060 4230 2110 4230
-Wire Wire Line
 	2160 4230 2160 4015
-Connection ~ 2060 4015
 Wire Wire Line
 	2060 4015 2060 4230
-Connection ~ 2160 4015
-Wire Wire Line
-	2160 4015 2160 4010
-Wire Wire Line
-	2110 4230 2110 4330
-Connection ~ 2110 4230
-Wire Wire Line
-	2110 4230 2160 4230
-$Comp
-L power:GND #PWR?
-U 1 1 5B92EDF1
-P 2110 4330
-F 0 "#PWR?" H 2110 4080 50  0001 C CNN
-F 1 "GND" H 2115 4157 50  0000 C CNN
-F 2 "" H 2110 4330 50  0001 C CNN
-F 3 "" H 2110 4330 50  0001 C CNN
-	1    2110 4330
-	1    0    0    -1
-$EndComp
-Text Label 5595 3465 3    50   ~ 0
-EN_RGB1
-Wire Wire Line
-	5595 3465 5595 3770
-Wire Wire Line
-	6265 3770 6265 3465
-Text Label 6265 3465 3    50   ~ 0
-EN_RGB2
-Wire Wire Line
-	6885 3770 6885 3470
-Text Label 6885 3470 3    50   ~ 0
-EN_RGB3
-Wire Wire Line
-	7555 3770 7555 3470
-Text Label 7555 3470 3    50   ~ 0
-EN_RGB4
+Wire Wire Line
+	6885 4070 6885 4165
 $EndSCHEMATC

Commit message: adding files to match the previous commit
Parts:
- C?: value C -> 10u
- C?: value C -> 0.1u
Connections:
- wire segments 121 -> 128
Changed lines of the file:
@@
 P 10090 1345
 F 0 "C?" H 10205 1391 50  0000 L CNN
-F 1 "C" H 10205 1300 50  0000 L CNN
+F 1 "10u" H 10205 1300 50  0000 L CNN
 F 2 "" H 10128 1195 50  0001 C CNN
 F 3 "~" H 10090 1345 50  0001 C CNN
@@
 P 10665 1345
 F 0 "C?" H 10780 1391 50  0000 L CNN
-F 1 "C" H 10780 1300 50  0000 L CNN
+F 1 "0.1u" H 10780 1300 50  0000 L CNN
 F 2 "" H 10703 1195 50  0001 C CNN
 F 3 "~" H 10665 1345 50  0001 C CNN
@@
 Wire Wire Line
 	6885 4070 6885 4165
+$Comp
+L power:GND #PWR?
+U 1 1 5BA1C59D
+P 10090 1585
+F 0 "#PWR?" H 10090 1335 50  0001 C CNN
+F 1 "GND" H 10095 1412 50  0000 C CNN
+F 2 "" H 10090 1585 50  0001 C CNN
+F 3 "" H 10090 1585 50  0001 C CNN
+	1    10090 1585
+	1    0    0    -1
+$EndComp
+Wire Wire Line
+	10090 1495 10090 1585
+$Comp
+L power:GND #PWR?
+U 1 1 5BA1FECE
+P 10665 1585
+F 0 "#PWR?" H 10665 1335 50  0001 C CNN
+F 1 "GND" H 10670 1412 50  0000 C CNN
+F 2 "" H 10665 1585 50  0001 C CNN
+F 3 "" H 10665 1585 50  0001 C CNN
+	1    10665 1585
+	1    0    0    -1
+$EndComp
+Wire Wire Line
+	10665 1495 10665 1585
+Wire Wire Line
+	2160 1600 2110 1600
+Wire Wire Line
+	2110 1600 2110 1500
+Connection ~ 2110 1600
+Wire Wire Line
+	2110 1600 2060 1600
+Wire Wire Line
+	2060 1600 2060 1815
+Wire Wire Line
+	2160 1815 2160 1600
+Text Label 2110 1500 0    50   ~ 0
+3V0
 $EndSCHEMATC
