File: HW/BSidesPDX_2018/BSidesPDX_2018.sch (KiCad schematic (older format))
At the start: 33 parts

Commit message: wired up ISP header, SAO I2C, and PWM
Parts:
- added J?: AVR-ISP-6, symbol Connector:AVR-ISP-6
Connections:
- net labels added: R_PWM__MISO, SCL_SCK, SDA_MOSI, ~RESET
- net labels removed: R_PWM, SCL, SDA
- wire segments 128 -> 149

Commit message: Wired, labeled, annotated charlieplex LEDs
Parts:
- removed D? (x6): LED, symbol Device:LED
- removed R? (x4): 100R, symbol Device:R
- added D? (x6): LED, symbol Device:LED
- added R3, R4, R? (x2): 100R, symbol Device:R
- gave numbers to parts that had none: 14
Connections:
- net labels added: ROW1, ROW2, ROW3, ROW4, ROW_1, ROW_2, ROW_3, ROW_4
- wire segments 149 -> 150

Commit message: Building BOM, added switches
Parts:
- added S? (x2): PTS645SM43SMTR92_LFS, digikey-footprints:Switch_Tactile_SMD_6x6mm_PTS645, symbol dk_Tactile-Switches:PTS645SM43SMTR92_LFS
- gave numbers to parts that had none: 18
Connections:
- net labels added: L_SWITCH, R_SWITCH
Changed lines of the file:
@@
 Sheet 1 1
 Title "BSidesPDX 2018 Badge"
-Date ""
+Date "2018-09-09"
 Rev "1.0"
-Comp ""
-Comment1 ""
-Comment2 ""
+Comp "https://github.com/pdxbadgers/badge-2018"
+Comment1 "Firmware, BOM, Schematic"
+Comment2 "@office_deskjet"
 Comment3 ""
 Comment4 ""
 $EndDescr
 $Comp
-L BSidesPDX_2018:Badgelife_shitty_connector X?
+L BSidesPDX_2018:Badgelife_shitty_connector X1
 U 1 1 5B8DDFA4
 P 1380 5940
-F 0 "X?" H 1480 6377 60  0000 C CNN
+F 0 "X1" H 1480 6377 60  0000 C CNN
 F 1 "Badgelife_shitty_connector" H 1470 6300 60  0000 C CNN
 F 2 "" H 1380 5940 60  0001 C CNN
@@
 $EndComp
 $Comp
-L Device:Battery_Cell BT?
+L Device:Battery_Cell BT1
 U 1 1 5B8DF1C7
 P 9300 1385
-F 0 "BT?" H 9418 1481 50  0000 L CNN
+F 0 "BT1" H 9418 1481 50  0000 L CNN
 F 1 "Battery_Cell" H 9418 1390 50  0000 L CNN
 F 2 "" V 9300 1445 50  0001 C CNN
@@
 SCL_SCK
 $Comp
-L BSidesPDX_2018:Badgelife_shitty_connector X?
+L BSidesPDX_2018:Badgelife_shitty_connector X2
 U 1 1 5B8E0671
 P 3000 5940
-F 0 "X?" H 3100 6377 60  0000 C CNN
+F 0 "X2" H 3100 6377 60  0000 C CNN
 F 1 "Badgelife_shitty_connector" H 3090 6300 60  0000 C CNN
 F 2 "" H 3000 5940 60  0001 C CNN
@@
 SCL_SCK
 $Comp
-L BSidesPDX_2018:Badgelife_shitty_connector X?
+L BSidesPDX_2018:Badgelife_shitty_connector X3
 U 1 1 5B8E1021
 P 4635 5940
-F 0 "X?" H 4735 6377 60  0000 C CNN
+F 0 "X3" H 4735 6377 60  0000 C CNN
 F 1 "Badgelife_shitty_connector" H 4725 6300 60  0000 C CNN
 F 2 "" H 4635 5940 60  0001 C CNN
@@
 SCL_SCK
 $Comp
-L BSidesPDX_2018:Badgelife_shitty_connector X?
+L BSidesPDX_2018:Badgelife_shitty_connector X4
 U 1 1 5B8E1038
 P 6365 5940
-F 0 "X?" H 6465 6377 60  0000 C CNN
+F 0 "X4" H 6465 6377 60  0000 C CNN
 F 1 "Badgelife_shitty_connector" H 6455 6300 60  0000 C CNN
 F 2 "" H 6365 5940 60  0001 C CNN
@@
 SCL_SCK
 $Comp
-L BSidesPDX_2018:Badgelife_shitty_connector X?
+L BSidesPDX_2018:Badgelife_shitty_connector X5
 U 1 1 5B8E1565
 P 8045 5940
-F 0 "X?" H 8145 6377 60  0000 C CNN
+F 0 "X5" H 8145 6377 60  0000 C CNN
 F 1 "Badgelife_shitty_connector" H 8135 6300 60  0000 C CNN
 F 2 "" H 8045 5940 60  0001 C CNN
@@
 EN_RGB4
 $Comp
-L Device:C C?
+L Device:C C1
 U 1 1 5B951E24
 P 10090 1345
-F 0 "C?" H 10205 1391 50  0000 L CNN
+F 0 "C1" H 10205 1391 50  0000 L CNN
 F 1 "10u" H 10205 1300 50  0000 L CNN
 F 2 "" H 10128 1195 50  0001 C CNN
@@
 $EndComp
 $Comp
-L Device:C C?
+L Device:C C2
 U 1 1 5B951F0C
 P 10665 1345
-F 0 "C?" H 10780 1391 50  0000 L CNN
+F 0 "C2" H 10780 1391 50  0000 L CNN
 F 1 "0.1u" H 10780 1300 50  0000 L CNN
 F 2 "" H 10703 1195 50  0001 C CNN
@@
 	7555 4070 7555 4165
 $Comp
-L MCU_Microchip_ATtiny:ATtiny861A-SU U?
+L MCU_Microchip_ATtiny:ATtiny861A-SU U1
 U 1 1 5B90B463
 P 2060 2915
-F 0 "U?" H 1430 2961 50  0000 R CNN
+F 0 "U1" H 1430 2961 50  0000 R CNN
 F 1 "ATTINY861-15XD " H 1430 2870 50  0000 R CNN
 F 2 "Package_SO:SOIC-20W_7.5x12.8mm_P1.27mm" H 2060 2915 50  0001 C CIN
@@
 	6885 4070 6885 4165
 $Comp
-L power:GND #PWR?
+L power:GND #PWR01
 U 1 1 5BA1C59D
 P 10090 1585
-F 0 "#PWR?" H 10090 1335 50  0001 C CNN
+F 0 "#PWR01" H 10090 1335 50  0001 C CNN
 F 1 "GND" H 10095 1412 50  0000 C CNN
 F 2 "" H 10090 1585 50  0001 C CNN
@@
 	10090 1495 10090 1585
 $Comp
-L power:GND #PWR?
+L power:GND #PWR02
 U 1 1 5BA1FECE
 P 10665 1585
-F 0 "#PWR?" H 10665 1335 50  0001 C CNN
+F 0 "#PWR02" H 10665 1335 50  0001 C CNN
 F 1 "GND" H 10670 1412 50  0000 C CNN
 F 2 "" H 10665 1585 50  0001 C CNN
@@
 3V0
 $Comp
-L Connector:AVR-ISP-6 J?
+L Connector:AVR-ISP-6 J1
 U 1 1 5BA3951F
 P 9905 2925
-F 0 "J?" H 9625 3021 50  0000 R CNN
+F 0 "J1" H 9625 3021 50  0000 R CNN
 F 1 "AVR-ISP-6" H 9625 2930 50  0000 R CNN
 F 2 "" V 9655 2975 50  0001 C CNN
@@
 3V0
 $Comp
-L power:GND #PWR?
+L power:GND #PWR03
 U 1 1 5BA88B3D
 P 9805 3415
-F 0 "#PWR?" H 9805 3165 50  0001 C CNN
+F 0 "#PWR03" H 9805 3165 50  0001 C CNN
 F 1 "GND" H 9810 3242 50  0000 C CNN
 F 2 "" H 9805 3415 50  0001 C CNN
@@
 ROW4
 $Comp
-L Device:LED D?
+L Device:LED D7
 U 1 1 5BB892DC
 P 5265 2130
-F 0 "D?" H 5256 2346 50  0000 C CNN
+F 0 "D7" H 5256 2346 50  0000 C CNN
 F 1 "LED" H 5256 2255 50  0000 C CNN
 F 2 "" H 5265 2130 50  0001 C CNN
@@
 $EndComp
 $Comp
-L Device:LED D?
+L Device:LED D9
 U 1 1 5BB892E2
 P 5265 2530
-F 0 "D?" H 5256 2746 50  0000 C CNN
+F 0 "D9" H 5256 2746 50  0000 C CNN
 F 1 "LED" H 5256 2655 50  0000 C CNN
 F 2 "" H 5265 2530 50  0001 C CNN
@@
 $EndComp
 $Comp
-L Device:LED D?
+L Device:LED D11
 U 1 1 5BB892E8
 P 5265 2930
-F 0 "D?" H 5256 3146 50  0000 C CNN
+F 0 "D11" H 5256 3146 50  0000 C CNN
 F 1 "LED" H 5256 3055 50  0000 C CNN
 F 2 "" H 5265 2930 50  0001 C CNN
@@
 Connection ~ 4985 2530
 $Comp
-L Device:LED D?
+L Device:LED D8
 U 1 1 5BB892FC
 P 6165 2130
-F 0 "D?" H 6156 2346 50  0000 C CNN
+F 0 "D8" H 6156 2346 50  0000 C CNN
 F 1 "LED" H 6156 2255 50  0000 C CNN
 F 2 "" H 6165 2130 50  0001 C CNN
@@
 $EndComp
 $Comp
-L Device:LED D?
+L Device:LED D10
 U 1 1 5BB89302
 P 6165 2530
-F 0 "D?" H 6156 2746 50  0000 C CNN
+F 0 "D10" H 6156 2746 50  0000 C CNN
 F 1 "LED" H 6156 2655 50  0000 C CNN
 F 2 "" H 6165 2530 50  0001 C CNN
@@
 $EndComp
 $Comp
-L Device:LED D?
+L Device:LED D12
 U 1 1 5BB89308
 P 6165 2930
-F 0 "D?" H 6156 3146 50  0000 C CNN
+F 0 "D12" H 6156 3146 50  0000 C CNN
 F 1 "LED" H 6156 3055 50  0000 C CNN
 F 2 "" H 6165 2930 50  0001 C CNN
@@
 	5885 1870 5885 2130
 $Comp
-L Device:R R?
+L Device:R R2
 U 1 1 5BBC9A88
 P 6820 1720
-F 0 "R?" H 6890 1766 50  0000 L CNN
+F 0 "R2" H 6890 1766 50  0000 L CNN
 F 1 "100R" H 6890 1675 50  0000 L CNN
 F 2 "" V 6750 1720 50  0001 C CNN
@@
 	6820 1385 6820 1570
 $Comp
-L Device:R R?
+L Device:R R1
 U 1 1 5BBC9A92
 P 7720 1720
-F 0 "R?" H 7790 1766 50  0000 L CNN
+F 0 "R1" H 7790 1766 50  0000 L CNN
 F 1 "100R" H 7790 1675 50  0000 L CNN
 F 2 "" V 7650 1720 50  0001 C CNN
@@
 Text Label 3315 2415 2    50   ~ 0
 ROW4
+$Comp
+L Graphic:Logo_Open_Hardware_Small #LOGO?
+U 1 1 5BBD132A
+P 10895 6865
+F 0 "#LOGO?" H 10895 7140 50  0001 C CNN
+F 1 "Logo_Open_Hardware_Small" H 10895 6640 50  0001 C CNN
+F 2 "" H 10895 6865 50  0001 C CNN
+F 3 "~" H 10895 6865 50  0001 C CNN
+	1    10895 6865
+	1    0    0    -1
+$EndComp
+$Comp
+L dk_Tactile-Switches:PTS645SM43SMTR92_LFS S?
+U 1 1 5BBD3F71
+P 9150 4245
+F 0 "S?" H 9150 4592 60  0000 C CNN
+F 1 "PTS645SM43SMTR92_LFS" H 9150 4486 60  0000 C CNN
+F 2 "digikey-footprints:Switch_Tactile_SMD_6x6mm_PTS645" H 9350 4445 60  0001 L CNN
+F 3 "https://www.ckswitches.com/media/1471/pts645.pdf" H 9350 4545 60  0001 L CNN
+F 4 "CKN9112CT-ND" H 9350 4645 60  0001 L CNN "Digi-Key_PN"
+F 5 "PTS645SM43SMTR92 LFS" H 9350 4745 60  0001 L CNN "MPN"
+F 6 "Switches" H 9350 4845 60  0001 L CNN "Category"
+F 7 "Tactile Switches" H 9350 4945 60  0001 L CNN "Family"
+F 8 "https://www.ckswitches.com/media/1471/pts645.pdf" H 9350 5045 60  0001 L CNN "DK_Datasheet_Link"
+F 9 "/product-detail/en/c-k/PTS645SM43SMTR92-LFS/CKN9112CT-ND/1146934" H 9350 5145 60  0001 L CNN "DK_Detail_Page"
+F 10 "SWITCH TACTILE SPST-NO 0.05A 12V" H 9350 5245 60  0001 L CNN "Description"
+F 11 "C&K" H 9350 5345 60  0001 L CNN "Manufacturer"
+F 12 "Active" H 9350 5445 60  0001 L CNN "Status"
+	1    9150 4245
+	1    0    0    -1
+$EndComp
+$Comp
+L dk_Tactile-Switches:PTS645SM43SMTR92_LFS S?
+U 1 1 5BBD4238
+P 10240 4145
+F 0 "S?" H 10240 4492 60  0000 C CNN
+F 1 "PTS645SM43SMTR92_LFS" H 10240 4386 60  0000 C CNN
+F 2 "digikey-footprints:Switch_Tactile_SMD_6x6mm_PTS645" H 10440 4345 60  0001 L CNN
+F 3 "https://www.ckswitches.com/media/1471/pts645.pdf" H 10440 4445 60  0001 L CNN
+F 4 "CKN9112CT-ND" H 10440 4545 60  0001 L CNN "Digi-Key_PN"
+F 5 "PTS645SM43SMTR92 LFS" H 10440 4645 60  0001 L CNN "MPN"
+F 6 "Switches" H 10440 4745 60  0001 L CNN "Category"
+F 7 "Tactile Switches" H 10440 4845 60  0001 L CNN "Family"
+F 8 "https://www.ckswitches.com/media/1471/pts645.pdf" H 10440 4945 60  0001 L CNN "DK_Datasheet_Link"
+F 9 "/product-detail/en/c-k/PTS645SM43SMTR92-LFS/CKN9112CT-ND/1146934" H 10440 5045 60  0001 L CNN "DK_Detail_Page"
+F 10 "SWITCH TACTILE SPST-NO 0.05A 12V" H 10440 5145 60  0001 L CNN "Description"
+F 11 "C&K" H 10440 5245 60  0001 L CNN "Manufacturer"
+F 12 "Active" H 10440 5345 60  0001 L CNN "Status"
+	1    10240 4145
+	1    0    0    -1
+$EndComp
+Text Label 3315 3415 2    50   ~ 0
+L_SWITCH
+Text Label 3315 3615 2    50   ~ 0
+R_SWITCH
 $EndSCHEMATC

Commit message: adding footprints
Parts:
- removed S?: PTS645SM43SMTR92_LFS, digikey-footprints:Switch_Tactile_SMD_6x6mm_PTS645, symbol dk_Tactile-Switches:PTS645SM43SMTR92_LFS
- added S2: PTS645SM43SMTR92_LFS, digikey-footprints:Switch_Tactile_SMD_6x6mm_PTS645, symbol dk_Tactile-Switches:PTS645SM43SMTR92_LFS
- D1, D10, D11, D12, D2, D3, D4, D5, D6, D7, D8, D9: value LED -> YLW_LED; footprint (none) -> BSidesPDX_2018:OSRAM_LED
- D101, D102, D103, D104: footprint (none) -> BSidesPDX_2018:RGB_LED
- J1: footprint (none) -> Pin_Headers:Pin_Header_Straight_2x03_Pitch2.54mm_SMD
- X1, X2, X3, X4, X5: footprint (none) -> BSidesPDX_2018:Badgelife-Shitty-2x2
- gave numbers to parts that had none: 1
Connections:
- wire segments 150 -> 172

Commit message: added a README for hardwre, updated footprints
Parts:
- C1: footprint (none) -> pkl_dipol:C_0805
- C2: footprint (none) -> pkl_dipol:C_0402
- R1, R101, R102, R103, R104, R2, R3, R4: footprint (none) -> pkl_dipol:R_0603
Changed lines of the file:
@@
 F 0 "R101" H 5665 3966 50  0000 L CNN
 F 1 "100R" H 5665 3875 50  0000 L CNN
-F 2 "" V 5525 3920 50  0001 C CNN
+F 2 "pkl_dipol:R_0603" V 5525 3920 50  0001 C CNN
 F 3 "~" H 5595 3920 50  0001 C CNN
 	1    5595 3920
@@
 F 0 "R102" H 6335 3966 50  0000 L CNN
 F 1 "100R" H 6335 3875 50  0000 L CNN
-F 2 "" V 6195 3920 50  0001 C CNN
+F 2 "pkl_dipol:R_0603" V 6195 3920 50  0001 C CNN
 F 3 "~" H 6265 3920 50  0001 C CNN
 	1    6265 3920
@@
 F 0 "R103" H 6955 3966 50  0000 L CNN
 F 1 "100R" H 6955 3875 50  0000 L CNN
-F 2 "" V 6815 3920 50  0001 C CNN
+F 2 "pkl_dipol:R_0603" V 6815 3920 50  0001 C CNN
 F 3 "~" H 6885 3920 50  0001 C CNN
 	1    6885 3920
@@
 F 0 "R104" H 7625 3966 50  0000 L CNN
 F 1 "100R" H 7625 3875 50  0000 L CNN
-F 2 "" V 7485 3920 50  0001 C CNN
+F 2 "pkl_dipol:R_0603" V 7485 3920 50  0001 C CNN
 F 3 "~" H 7555 3920 50  0001 C CNN
 	1    7555 3920
@@
 F 0 "C1" H 10205 1391 50  0000 L CNN
 F 1 "10u" H 10205 1300 50  0000 L CNN
-F 2 "" H 10128 1195 50  0001 C CNN
+F 2 "pkl_dipol:C_0805" H 10128 1195 50  0001 C CNN
 F 3 "~" H 10090 1345 50  0001 C CNN
 	1    10090 1345
@@
 F 0 "C2" H 10780 1391 50  0000 L CNN
 F 1 "0.1u" H 10780 1300 50  0000 L CNN
-F 2 "" H 10703 1195 50  0001 C CNN
+F 2 "pkl_dipol:C_0402" H 10703 1195 50  0001 C CNN
 F 3 "~" H 10665 1345 50  0001 C CNN
 	1    10665 1345
@@
 F 0 "R4" H 5055 1766 50  0000 L CNN
 F 1 "100R" H 5055 1675 50  0000 L CNN
-F 2 "" V 4915 1720 50  0001 C CNN
+F 2 "pkl_dipol:R_0603" V 4915 1720 50  0001 C CNN
 F 3 "~" H 4985 1720 50  0001 C CNN
 	1    4985 1720
@@
 F 0 "R3" H 5955 1766 50  0000 L CNN
 F 1 "100R" H 5955 1675 50  0000 L CNN
-F 2 "" V 5815 1720 50  0001 C CNN
+F 2 "pkl_dipol:R_0603" V 5815 1720 50  0001 C CNN
 F 3 "~" H 5885 1720 50  0001 C CNN
 	1    5885 1720
@@
 F 0 "R2" H 6890 1766 50  0000 L CNN
 F 1 "100R" H 6890 1675 50  0000 L CNN
-F 2 "" V 6750 1720 50  0001 C CNN
+F 2 "pkl_dipol:R_0603" V 6750 1720 50  0001 C CNN
 F 3 "~" H 6820 1720 50  0001 C CNN
 	1    6820 1720
@@
 F 0 "R1" H 7790 1766 50  0000 L CNN
 F 1 "100R" H 7790 1675 50  0000 L CNN
-F 2 "" V 7650 1720 50  0001 C CNN
+F 2 "pkl_dipol:R_0603" V 7650 1720 50  0001 C CNN
 F 3 "~" H 7720 1720 50  0001 C CNN
 	1    7720 1720

Commit message: Added LED and battery retainer datasheets. Added footprint for battery retainer. Update footprints in schematic.
Parts:
- BT1: footprint (none) -> BSidesPDX_2018:CR2030_Retainer
Changed lines of the file:
@@
 F 0 "BT1" H 9418 1481 50  0000 L CNN
 F 1 "Battery_Cell" H 9418 1390 50  0000 L CNN
-F 2 "" V 9300 1445 50  0001 C CNN
+F 2 "BSidesPDX_2018:CR2030_Retainer" V 9300 1445 50  0001 C CNN
 F 3 "~" V 9300 1445 50  0001 C CNN
 	1    9300 1385

Commit message: added press fit SAO connector, updated SAO footprints, added schematic for USB connecotr
Parts:
- added J2: USB_B_Micro, symbol Connector:USB_B_Micro
- added R5, R6: 22R, symbol Device:R
- X1, X2, X3, X4, X5: footprint BSidesPDX_2018:Badgelife-Shitty-2x2 -> BSidesPDX_2018:PRESS_FIT_SAO_CNX
Connections:
- wire segments 172 -> 185
Other:
- moved on the sheet: U1
Changed lines of the file:
@@
 F 0 "X1" H 1480 6392 60  0000 C CNN
 F 1 "Badgelife_shitty_connector" H 1470 6315 60  0000 C CNN
-F 2 "BSidesPDX_2018:Badgelife-Shitty-2x2" H 1380 5955 60  0001 C CNN
+F 2 "BSidesPDX_2018:PRESS_FIT_SAO_CNX" H 1380 5955 60  0001 C CNN
 F 3 "" H 1380 5955 60  0001 C CNN
 	1    1380 5955
@@
 F 0 "X2" H 3100 6392 60  0000 C CNN
 F 1 "Badgelife_shitty_connector" H 3090 6315 60  0000 C CNN
-F 2 "BSidesPDX_2018:Badgelife-Shitty-2x2" H 3000 5955 60  0001 C CNN
+F 2 "BSidesPDX_2018:PRESS_FIT_SAO_CNX" H 3000 5955 60  0001 C CNN
 F 3 "" H 3000 5955 60  0001 C CNN
 	1    3000 5955
@@
 F 0 "X3" H 4735 6392 60  0000 C CNN
 F 1 "Badgelife_shitty_connector" H 4725 6315 60  0000 C CNN
-F 2 "BSidesPDX_2018:Badgelife-Shitty-2x2" H 4635 5955 60  0001 C CNN
+F 2 "BSidesPDX_2018:PRESS_FIT_SAO_CNX" H 4635 5955 60  0001 C CNN
 F 3 "" H 4635 5955 60  0001 C CNN
 	1    4635 5955
@@
 F 0 "X4" H 6465 6392 60  0000 C CNN
 F 1 "Badgelife_shitty_connector" H 6455 6315 60  0000 C CNN
-F 2 "BSidesPDX_2018:Badgelife-Shitty-2x2" H 6365 5955 60  0001 C CNN
+F 2 "BSidesPDX_2018:PRESS_FIT_SAO_CNX" H 6365 5955 60  0001 C CNN
 F 3 "" H 6365 5955 60  0001 C CNN
 	1    6365 5955
@@
 F 0 "X5" H 8145 6392 60  0000 C CNN
 F 1 "Badgelife_shitty_connector" H 8135 6315 60  0000 C CNN
-F 2 "BSidesPDX_2018:Badgelife-Shitty-2x2" H 8045 5955 60  0001 C CNN
+F 2 "BSidesPDX_2018:PRESS_FIT_SAO_CNX" H 8045 5955 60  0001 C CNN
 F 3 "" H 8045 5955 60  0001 C CNN
 	1    8045 5955
@@
 Connection ~ 7720 2530
 Wire Wire Line
-	2060 4230 2110 4230
-Wire Wire Line
-	2110 4230 2110 4330
-Connection ~ 2110 4230
-Wire Wire Line
-	2110 4230 2160 4230
+	1950 3760 2000 3760
+Wire Wire Line
+	2000 3760 2000 3860
+Connection ~ 2000 3760
+Wire Wire Line
+	2000 3760 2050 3760
 $Comp
 L power:GND #PWR0107
 U 1 1 5B92EDF1
-P 2110 4330
-F 0 "#PWR0107" H 2110 4080 50  0001 C CNN
-F 1 "GND" H 2115 4157 50  0000 C CNN
-F 2 "" H 2110 4330 50  0001 C CNN
-F 3 "" H 2110 4330 50  0001 C CNN
-	1    2110 4330
+P 2000 3860
+F 0 "#PWR0107" H 2000 3610 50  0001 C CNN
+F 1 "GND" H 2005 3687 50  0000 C CNN
+F 2 "" H 2000 3860 50  0001 C CNN
+F 3 "" H 2000 3860 50  0001 C CNN
+	1    2000 3860
 	1    0    0    -1
 $EndComp
@@
 L MCU_Microchip_ATtiny:ATtiny861A-SU U1
 U 1 1 5B90B463
-P 2060 2915
-F 0 "U1" H 1430 2961 50  0000 R CNN
-F 1 "ATTINY861-15XD " H 1430 2870 50  0000 R CNN
-F 2 "Package_SO:SOIC-20W_7.5x12.8mm_P1.27mm" H 2060 2915 50  0001 C CIN
-F 3 "http://ww1.microchip.com/downloads/en/DeviceDoc/doc8197.pdf" H 2060 2915 50  0001 C CNN
-	1    2060 2915
-	1    0    0    -1
-$EndComp
-Wire Wire Line
-	2160 4230 2160 4015
-Wire Wire Line
-	2060 4015 2060 4230
+P 1950 2445
+F 0 "U1" H 1320 2491 50  0000 R CNN
+F 1 "ATTINY861-15XD " H 1320 2400 50  0000 R CNN
+F 2 "Package_SO:SOIC-20W_7.5x12.8mm_P1.27mm" H 1950 2445 50  0001 C CIN
+F 3 "http://ww1.microchip.com/downloads/en/DeviceDoc/doc8197.pdf" H 1950 2445 50  0001 C CNN
+	1    1950 2445
+	1    0    0    -1
+$EndComp
+Wire Wire Line
+	2050 3760 2050 3545
+Wire Wire Line
+	1950 3545 1950 3760
 Wire Wire Line
 	6885 4070 6885 4165
@@
 	10665 1495 10665 1585
 Wire Wire Line
-	2160 1600 2110 1600
-Wire Wire Line
-	2110 1600 2110 1500
-Connection ~ 2110 1600
-Wire Wire Line
-	2110 1600 2060 1600
-Wire Wire Line
-	2060 1600 2060 1815
-Wire Wire Line
-	2160 1815 2160 1600
-Text Label 2110 1500 0    50   ~ 0
+	2050 1130 2000 1130
+Wire Wire Line
+	2000 1130 2000 1030
+Connection ~ 2000 1130
+Wire Wire Line
+	2000 1130 1950 1130
+Wire Wire Line
+	1950 1130 1950 1345
+Wire Wire Line
+	2050 1345 2050 1130
+Text Label 2000 1030 0    50   ~ 0
 3V0
 $Comp
@@
 $EndComp
 Wire Wire Line
-	2760 3115 3315 3115
-Wire Wire Line
-	2760 3315 3315 3315
-Wire Wire Line
-	2760 3515 3315 3515
-Text Label 3315 3115 2    50   ~ 0
+	2650 2645 3205 2645
+Wire Wire Line
+	2650 2845 3205 2845
+Wire Wire Line
+	2650 3045 3205 3045
+Text Label 3205 2645 2    50   ~ 0
 R_PWM__MISO
 Wire Wire Line
@@
 Wire Wire Line
 	7455 4815 7455 5180
-Text Label 3315 3315 2    50   ~ 0
+Text Label 3205 2845 2    50   ~ 0
 G_PWM
-Text Label 3315 3515 2    50   ~ 0
+Text Label 3205 3045 2    50   ~ 0
 B_PWM
 Wire Wire Line
-	2760 3615 3315 3615
-Wire Wire Line
-	2760 3415 3315 3415
+	2650 3145 3205 3145
+Wire Wire Line
+	2650 2945 3205 2945
 Text Label 9805 2275 0    50   ~ 0
 3V0
@@
 	9805 3325 9805 3415
 Wire Wire Line
-	2760 3715 3315 3715
-Wire Wire Line
-	2760 2115 3315 2115
-Wire Wire Line
-	2760 2215 3315 2215
-Wire Wire Line
-	2760 2315 3315 2315
-Wire Wire Line
-	2760 2415 3315 2415
-Wire Wire Line
-	2760 2515 3315 2515
-Wire Wire Line
-	2760 2615 3315 2615
-Wire Wire Line
-	2760 2715 3315 2715
-Wire Wire Line
-	2760 3215 3315 3215
-Text Label 3315 3015 2    50   ~ 0
+	2650 3245 3205 3245
+Wire Wire Line
+	2650 1645 3205 1645
+Wire Wire Line
+	2650 1745 3205 1745
+Wire Wire Line
+	2650 1845 3205 1845
+Wire Wire Line
+	2650 1945 3205 1945
+Wire Wire Line
+	2650 2045 3205 2045
+Wire Wire Line
+	2650 2145 3205 2145
+Wire Wire Line
+	2650 2245 3205 2245
+Wire Wire Line
+	2650 2745 3205 2745
+Text Label 3205 2545 2    50   ~ 0
 SDA_MOSI
 Wire Wire Line
@@
 Text Label 10455 2825 0    50   ~ 0
 SDA_MOSI
-Text Label 3315 3715 2    50   ~ 0
+Text Label 3205 3245 2    50   ~ 0
 ~RESET
 Text Label 10455 3025 0    50   ~ 0
@@
 SCL_SCK
 Wire Wire Line
-	2760 3015 3315 3015
-Text Label 3315 3215 2    50   ~ 0
+	2650 2545 3205 2545
+Text Label 3205 2745 2    50   ~ 0
 SCL_SCK
 Wire Wire Line
-	2760 2815 3315 2815
-Text Label 3315 2515 2    50   ~ 0
+	2650 2345 3205 2345
+Text Label 3205 2045 2    50   ~ 0
 EN_RGB1
-Text Label 3315 2615 2    50   ~ 0
+Text Label 3205 2145 2    50   ~ 0
 EN_RGB2
-Text Label 3315 2715 2    50   ~ 0
+Text Label 3205 2245 2    50   ~ 0
 EN_RGB3
-Text Label 3315 2815 2    50   ~ 0
+Text Label 3205 2345 2    50   ~ 0
 EN_RGB4
 Wire Wire Line
@@
 Connection ~ 6820 2130
 Connection ~ 7720 2130
-Text Label 3315 2115 2    50   ~ 0
+Text Label 3205 1645 2    50   ~ 0
 ROW1
-Text Label 3315 2215 2    50   ~ 0
+Text Label 3205 1745 2    50   ~ 0
 ROW2
-Text Label 3315 2315 2    50   ~ 0
+Text Label 3205 1845 2    50   ~ 0
 ROW3
-Text Label 3315 2415 2    50   ~ 0
+Text Label 3205 1945 2    50   ~ 0
 ROW4
 $Comp
@@
 	1    0    0    -1
 $EndComp
-Text Label 3315 3415 2    50   ~ 0
+Text Label 3205 2945 2    50   ~ 0
 L_SWITCH
-Text Label 3315 3615 2    50   ~ 0
+Text Label 3205 3145 2    50   ~ 0
 R_SWITCH
 Wire Wire Line
@@
 Wire Wire Line
 	9805 2425 9805 2275
+$Comp
+L Connector:USB_B_Micro J2
+U 1 1 5B8FAB2D
+P 2000 4690
+F 0 "J2" H 2055 5157 50  0000 C CNN
+F 1 "USB_B_Micro" H 2055 5066 50  0000 C CNN
+F 2 "" H 2150 4640 50  0001 C CNN
+F 3 "~" H 2150 4640 50  0001 C CNN
+	1    2000 4690
+	1    0    0    -1
+$EndComp
+Wire Wire Line
+	2300 4490 2500 4490
+Wire Wire Line
+	2300 4690 2420 4690
+Wire Wire Line
+	2300 4890 2360 4890
+$Comp
+L power:GND #PWR04
+U 1 1 5B94549A
+P 2140 5160
+F 0 "#PWR04" H 2140 4910 50  0001 C CNN
+F 1 "GND" H 2145 4987 50  0000 C CNN
+F 2 "" H 2140 5160 50  0001 C CNN
+F 3 "" H 2140 5160 50  0001 C CNN
+	1    2140 5160
+	1    0    0    -1
+$EndComp
+Text Label 2500 4490 2    50   ~ 0
+3V0
+Wire Wire Line
+	2360 4890 2360 5090
+Wire Wire Line
+	2360 5090 2140 5090
+Connection ~ 2000 5090
+Wire Wire Line
+	2140 5160 2140 5090
+Wire Wire Line
+	1900 5090 2000 5090
+Connection ~ 2140 5090
+Wire Wire Line
+	2140 5090 2000 5090
+$Comp
+L Device:R R5
+U 1 1 5B986B50
+P 2570 4690
+F 0 "R5" V 2490 4690 50  0000 C CNN
+F 1 "22R" V 2570 4690 50  0000 C CNN
+F 2 "" V 2500 4690 50  0001 C CNN
+F 3 "~" H 2570 4690 50  0001 C CNN
+	1    2570 4690
+	0    1    1    0
+$EndComp
+Wire Wire Line
+	2300 4790 2720 4790
+$Comp
+L Device:R R6
+U 1 1 5B98F378
+P 2870 4790
+F 0 "R6" V 2940 4790 50  0000 C CNN
+F 1 "22R" V 2860 4790 50  0000 C CNN
+F 2 "" V 2800 4790 50  0001 C CNN
+F 3 "~" H 2870 4790 50  0001 C CNN
+	1    2870 4790
+	0    -1   -1   0
+$EndComp
+Wire Wire Line
+	2720 4690 2780 4690
+Wire Wire Line
+	3020 4790 3090 4790
+Wire Wire Line
+	2780 4270 2780 4690
+Wire Wire Line
+	3090 4270 3090 4790
+Text Label 2780 4270 3    50   ~ 0
+L_SWITCH
+Text Label 3090 4270 3    50   ~ 0
+R_SWITCH
 $EndSCHEMATC

Commit message: Corrected footprint for MCU. Updated USB parts
Parts:
- J2: footprint (none) -> Connector_USB:USB_Micro-B_Molex_47346-0001
- R5, R6: value 22R -> DNP
- U1: footprint Package_SO:SOIC-20W_7.5x12.8mm_P1.27mm -> Package_SO:TSSOP-20_4.4x6.5mm_P0.65mm
Changed lines of the file:
@@
 F 0 "U1" H 1320 2491 50  0000 R CNN
 F 1 "ATTINY861-15XD " H 1320 2400 50  0000 R CNN
-F 2 "Package_SO:SOIC-20W_7.5x12.8mm_P1.27mm" H 1950 2445 50  0001 C CIN
+F 2 "Package_SO:TSSOP-20_4.4x6.5mm_P0.65mm" H 1950 2445 50  0001 C CIN
 F 3 "http://ww1.microchip.com/downloads/en/DeviceDoc/doc8197.pdf" H 1950 2445 50  0001 C CNN
 	1    1950 2445
@@
 F 0 "J2" H 2055 5157 50  0000 C CNN
 F 1 "USB_B_Micro" H 2055 5066 50  0000 C CNN
-F 2 "" H 2150 4640 50  0001 C CNN
+F 2 "Connector_USB:USB_Micro-B_Molex_47346-0001" H 2150 4640 50  0001 C CNN
 F 3 "~" H 2150 4640 50  0001 C CNN
 	1    2000 4690
@@
 P 2570 4690
 F 0 "R5" V 2490 4690 50  0000 C CNN
-F 1 "22R" V 2570 4690 50  0000 C CNN
+F 1 "DNP" V 2570 4690 50  0000 C CNN
 F 2 "" V 2500 4690 50  0001 C CNN
 F 3 "~" H 2570 4690 50  0001 C CNN
@@
 P 2870 4790
 F 0 "R6" V 2940 4790 50  0000 C CNN
-F 1 "22R" V 2860 4790 50  0000 C CNN
+F 1 "DNP" V 2860 4790 50  0000 C CNN
 F 2 "" V 2800 4790 50  0001 C CNN
 F 3 "~" H 2870 4790 50  0001 C CNN
