File: HW/BSidesPDX_2018/BSidesPDX_2018.sch (KiCad schematic (older format))
At the start: 39 parts, among them J1 AVR-ISP-6, J2 USB_B_Micro, U1 ATTINY861-15XD, X1 Badgelife_shitty_connector, X2 Badgelife_shitty_connector, X3 Badgelife_shitty_connector, X4 Badgelife_shitty_connector, X5 Badgelife_shitty_connector

Commit message: removed USB connector, it will move to addon
Parts:
- removed J2: USB_B_Micro, Connector_USB:USB_Micro-B_Molex_47346-0001, symbol Connector:USB_B_Micro
- removed R5, R6: DNP, symbol Device:R
Connections:
- wire segments 185 -> 172
Changed lines of the file:
@@
 Wire Wire Line
 	9805 2425 9805 2275
-$Comp
-L Connector:USB_B_Micro J2
-U 1 1 5B8FAB2D
-P 2000 4690
-F 0 "J2" H 2055 5157 50  0000 C CNN
-F 1 "USB_B_Micro" H 2055 5066 50  0000 C CNN
-F 2 "Connector_USB:USB_Micro-B_Molex_47346-0001" H 2150 4640 50  0001 C CNN
-F 3 "~" H 2150 4640 50  0001 C CNN
-	1    2000 4690
-	1    0    0    -1
-$EndComp
-Wire Wire Line
-	2300 4490 2500 4490
-Wire Wire Line
-	2300 4690 2420 4690
-Wire Wire Line
-	2300 4890 2360 4890
-$Comp
-L power:GND #PWR04
-U 1 1 5B94549A
-P 2140 5160
-F 0 "#PWR04" H 2140 4910 50  0001 C CNN
-F 1 "GND" H 2145 4987 50  0000 C CNN
-F 2 "" H 2140 5160 50  0001 C CNN
-F 3 "" H 2140 5160 50  0001 C CNN
-	1    2140 5160
-	1    0    0    -1
-$EndComp
-Text Label 2500 4490 2    50   ~ 0
-3V0
-Wire Wire Line
-	2360 4890 2360 5090
-Wire Wire Line
-	2360 5090 2140 5090
-Connection ~ 2000 5090
-Wire Wire Line
-	2140 5160 2140 5090
-Wire Wire Line
-	1900 5090 2000 5090
-Connection ~ 2140 5090
-Wire Wire Line
-	2140 5090 2000 5090
-$Comp
-L Device:R R5
-U 1 1 5B986B50
-P 2570 4690
-F 0 "R5" V 2490 4690 50  0000 C CNN
-F 1 "DNP" V 2570 4690 50  0000 C CNN
-F 2 "" V 2500 4690 50  0001 C CNN
-F 3 "~" H 2570 4690 50  0001 C CNN
-	1    2570 4690
-	0    1    1    0
-$EndComp
-Wire Wire Line
-	2300 4790 2720 4790
-$Comp
-L Device:R R6
-U 1 1 5B98F378
-P 2870 4790
-F 0 "R6" V 2940 4790 50  0000 C CNN
-F 1 "DNP" V 2860 4790 50  0000 C CNN
-F 2 "" V 2800 4790 50  0001 C CNN
-F 3 "~" H 2870 4790 50  0001 C CNN
-	1    2870 4790
-	0    -1   -1   0
-$EndComp
-Wire Wire Line
-	2720 4690 2780 4690
-Wire Wire Line
-	3020 4790 3090 4790
-Wire Wire Line
-	2780 4270 2780 4690
-Wire Wire Line
-	3090 4270 3090 4790
-Text Label 2780 4270 3    50   ~ 0
-L_SWITCH
-Text Label 3090 4270 3    50   ~ 0
-R_SWITCH
 $EndSCHEMATC

Commit message: added foot print for programming header. Footpints are now assigned.
Parts:
- J1: footprint Pin_Headers:Pin_Header_Straight_2x03_Pitch2.54mm_SMD -> BSidesPDX_2018:AVR_ISP_2x3_P2.54mm_SMD
Changed lines of the file:
@@
 F 0 "J1" H 9625 3021 50  0000 R CNN
 F 1 "AVR-ISP-6" H 9625 2930 50  0000 R CNN
-F 2 "Pin_Headers:Pin_Header_Straight_2x03_Pitch2.54mm_SMD" V 9655 2975 50  0001 C CNN
+F 2 "BSidesPDX_2018:AVR_ISP_2x3_P2.54mm_SMD" V 9655 2975 50  0001 C CNN
 F 3 " ~" H 8630 2375 50  0001 C CNN
 	1    9905 2925

Commit message: removed bottom SAO, Added USB back, updated library paths
Parts:
- removed X5: Badgelife_shitty_connector, BSidesPDX_2018:PRESS_FIT_SAO_CNX, symbol BSidesPDX_2018:Badgelife_shitty_connector
- added J2: USB_B_Micro, Connector_USB:USB_Micro-B_Molex_47346-0001, symbol Connector:USB_B_Micro
- added R5, R6: 51, symbol Device:R
- J1: footprint BSidesPDX_2018:AVR_ISP_2x3_P2.54mm_SMD -> Pin_Headers:Pin_Header_Straight_2x03_Pitch2.54mm_SMD
Connections:
- net labels added: SCL_SCK_D-, SDA_MOSI_D+
- net labels removed: SCL_SCK, SDA_MOSI
- wire segments 172 -> 175

Commit message: updated BOM, but missing resistor links. Updated Footprints
Parts:
- added R7: 1K, pkl_dipol:R_0603, symbol Device:R
- R5, R6: value 51 -> 51R; footprint (none) -> pkl_dipol:R_0603
Connections:
- wire segments 175 -> 177
Changed lines of the file:
@@
 P 2570 4690
 F 0 "R5" V 2490 4690 50  0000 C CNN
-F 1 "51" V 2570 4690 50  0000 C CNN
-F 2 "" V 2500 4690 50  0001 C CNN
+F 1 "51R" V 2570 4690 50  0000 C CNN
+F 2 "pkl_dipol:R_0603" V 2500 4690 50  0001 C CNN
 F 3 "~" H 2570 4690 50  0001 C CNN
 	1    2570 4690
@@
 P 2870 4790
 F 0 "R6" V 2780 4790 50  0000 C CNN
-F 1 "51" V 2860 4790 50  0000 C CNN
-F 2 "" V 2800 4790 50  0001 C CNN
+F 1 "51R" V 2860 4790 50  0000 C CNN
+F 2 "pkl_dipol:R_0603" V 2800 4790 50  0001 C CNN
 F 3 "~" H 2870 4790 50  0001 C CNN
 	1    2870 4790
@@
 SCL_SCK_D-
 Wire Wire Line
-	3020 4790 3470 4790
+	2720 4690 3470 4690
+$Comp
+L Device:R R7
+U 1 1 5B94AAC6
+P 3610 4430
+F 0 "R7" H 3680 4476 50  0000 L CNN
+F 1 "1K" H 3680 4385 50  0000 L CNN
+F 2 "pkl_dipol:R_0603" V 3540 4430 50  0001 C CNN
+F 3 "~" H 3610 4430 50  0001 C CNN
+	1    3610 4430
+	1    0    0    -1
+$EndComp
 Wire Wire Line
-	2720 4690 3470 4690
+	3610 4280 3610 4070
+Text Label 3610 4070 0    50   ~ 0
+3V0
+Wire Wire Line
+	3610 4790 3610 4580
+Wire Wire Line
+	3020 4790 3610 4790
 $EndSCHEMATC

Commit message: Updated BOM USB connector, added USB footprint, updated ISP footprint, assigned footprints
Parts:
- J1: footprint Pin_Headers:Pin_Header_Straight_2x03_Pitch2.54mm_SMD -> BSidesPDX_2018:AVR_ISP_2x3_P2.54mm_SMD
- J2: footprint Connector_USB:USB_Micro-B_Molex_47346-0001 -> BSidesPDX_2018:USB_B_Micro
Changed lines of the file:
@@
 F 0 "J1" H 9625 3021 50  0000 R CNN
 F 1 "AVR-ISP-6" H 9625 2930 50  0000 R CNN
-F 2 "Pin_Headers:Pin_Header_Straight_2x03_Pitch2.54mm_SMD" V 9655 2975 50  0001 C CNN
+F 2 "BSidesPDX_2018:AVR_ISP_2x3_P2.54mm_SMD" V 9655 2975 50  0001 C CNN
 F 3 " ~" H 8630 2375 50  0001 C CNN
 	1    9905 2925
@@
 F 0 "J2" H 2055 5157 50  0000 C CNN
 F 1 "USB_B_Micro" H 2055 5066 50  0000 C CNN
-F 2 "Connector_USB:USB_Micro-B_Molex_47346-0001" H 2150 4640 50  0001 C CNN
+F 2 "BSidesPDX_2018:USB_B_Micro" H 2150 4640 50  0001 C CNN
 F 3 "~" H 2150 4640 50  0001 C CNN
 	1    2000 4690

Commit message: Layout work, added Datasheet for USB connector, fixed OSRAM_LED footprint, Fixed AVR ISP footprint.
Connections:
- net labels added: D+, D-
Changed lines of the file:
@@
 Wire Wire Line
 	3020 4790 3610 4790
+Text Label 2320 4690 0    50   ~ 0
+D+
+Text Label 2320 4790 0    50   ~ 0
+D-
 $EndSCHEMATC

Commit message: changed library settings, changed charliplexing circuit, fixed USB resistor
Connections:
- wire segments 177 -> 178
Changed lines of the file:
@@
 	8150 2930 8500 2930
 Text Label 8500 2130 2    50   ~ 0
-ROW2
+ROW_2
 Wire Wire Line
 	8150 2530 8500 2530
@@
 	8150 2130 8500 2130
 Text Label 8500 2530 2    50   ~ 0
-ROW3
+ROW_3
 Text Label 8500 2930 2    50   ~ 0
-ROW4
+ROW_4
 Wire Wire Line
 	7250 2930 7600 2930
 Text Label 7600 2130 2    50   ~ 0
-ROW1
+ROW_1
 Wire Wire Line
 	7250 2530 7600 2530
@@
 	7250 2130 7600 2130
 Text Label 7600 2530 2    50   ~ 0
-ROW3
+ROW_3
 Text Label 7600 2930 2    50   ~ 0
-ROW4
+ROW_4
 $Comp
 L Device:LED D7
@@
 	6315 2930 6665 2930
 Text Label 6665 2130 2    50   ~ 0
-ROW1
+ROW_1
 Wire Wire Line
 	6315 2530 6665 2530
@@
 	6315 2130 6665 2130
 Text Label 6665 2530 2    50   ~ 0
-ROW2
+ROW_2
 Text Label 6665 2930 2    50   ~ 0
-ROW4
+ROW_4
 Wire Wire Line
 	5415 2930 5765 2930
 Text Label 5765 2130 2    50   ~ 0
-ROW1
+ROW_1
 Wire Wire Line
 	5415 2530 5765 2530
@@
 	5415 2130 5765 2130
 Text Label 5765 2530 2    50   ~ 0
-ROW2
+ROW_2
 Text Label 5765 2930 2    50   ~ 0
-ROW3
+ROW_3
 Text Label 4985 1385 3    50   ~ 0
 ROW4
@@
 $EndComp
 Wire Wire Line
-	2300 4790 2720 4790
+	2300 4790 2840 4790
 $Comp
 L Device:R R6
 U 1 1 5B98F378
-P 2870 4790
-F 0 "R6" V 2780 4790 50  0000 C CNN
-F 1 "51R" V 2860 4790 50  0000 C CNN
-F 2 "pkl_dipol:R_0603" V 2800 4790 50  0001 C CNN
-F 3 "~" H 2870 4790 50  0001 C CNN
-	1    2870 4790
+P 3085 4790
+F 0 "R6" V 2995 4790 50  0000 C CNN
+F 1 "51R" V 3075 4790 50  0000 C CNN
+F 2 "pkl_dipol:R_0603" V 3015 4790 50  0001 C CNN
+F 3 "~" H 3085 4790 50  0001 C CNN
+	1    3085 4790
 	0    -1   -1   0
 $EndComp
-Text Label 3470 4690 2    50   ~ 0
+Text Label 3695 4690 2    50   ~ 0
 SDA_MOSI_D+
-Text Label 3470 4790 2    50   ~ 0
+Text Label 3700 4790 2    50   ~ 0
 SCL_SCK_D-
 Wire Wire Line
-	2720 4690 3470 4690
+	2720 4690 3695 4690
 $Comp
 L Device:R R7
 U 1 1 5B94AAC6
-P 3610 4430
-F 0 "R7" H 3680 4476 50  0000 L CNN
-F 1 "1K" H 3680 4385 50  0000 L CNN
-F 2 "pkl_dipol:R_0603" V 3540 4430 50  0001 C CNN
-F 3 "~" H 3610 4430 50  0001 C CNN
-	1    3610 4430
-	1    0    0    -1
-$EndComp
-Wire Wire Line
-	3610 4280 3610 4070
-Text Label 3610 4070 0    50   ~ 0
+P 2840 4430
+F 0 "R7" H 2910 4476 50  0000 L CNN
+F 1 "1K" H 2910 4385 50  0000 L CNN
+F 2 "pkl_dipol:R_0603" V 2770 4430 50  0001 C CNN
+F 3 "~" H 2840 4430 50  0001 C CNN
+	1    2840 4430
+	1    0    0    -1
+$EndComp
+Wire Wire Line
+	2840 4280 2840 4060
+Text Label 2840 4060 0    50   ~ 0
 3V0
-Wire Wire Line
-	3610 4790 3610 4580
-Wire Wire Line
-	3020 4790 3610 4790
 Text Label 2320 4690 0    50   ~ 0
 D+
 Text Label 2320 4790 0    50   ~ 0
 D-
+Wire Wire Line
+	3235 4790 3700 4790
+Wire Wire Line
+	2840 4790 2840 4580
+Connection ~ 2840 4790
+Wire Wire Line
+	2840 4790 2935 4790
 $EndSCHEMATC

Commit message: Moved foot prints from libraries to locally.
Parts:
- C1: footprint pkl_dipol:C_0805 -> BSidesPDX_2018:C_0805
- C2: footprint pkl_dipol:C_0402 -> BSidesPDX_2018:C_0603
- R1, R101, R102, R103, R104, R2, R3, R4, R5, R6, R7: footprint pkl_dipol:R_0603 -> BSidesPDX_2018:C_0603
- S1, S2: footprint digikey-footprints:Switch_Tactile_SMD_6x6mm_PTS645 -> BSidesPDX_2018:Switch_Tactile_SMD_6x6mm_PTS645
Changed lines of the file:
@@
 F 0 "R101" H 5665 3966 50  0000 L CNN
 F 1 "100R" H 5665 3875 50  0000 L CNN
-F 2 "pkl_dipol:R_0603" V 5525 3920 50  0001 C CNN
+F 2 "BSidesPDX_2018:C_0603" V 5525 3920 50  0001 C CNN
 F 3 "~" H 5595 3920 50  0001 C CNN
 	1    5595 3920
@@
 F 0 "R102" H 6335 3966 50  0000 L CNN
 F 1 "100R" H 6335 3875 50  0000 L CNN
-F 2 "pkl_dipol:R_0603" V 6195 3920 50  0001 C CNN
+F 2 "BSidesPDX_2018:C_0603" V 6195 3920 50  0001 C CNN
 F 3 "~" H 6265 3920 50  0001 C CNN
 	1    6265 3920
@@
 F 0 "R103" H 6955 3966 50  0000 L CNN
 F 1 "100R" H 6955 3875 50  0000 L CNN
-F 2 "pkl_dipol:R_0603" V 6815 3920 50  0001 C CNN
+F 2 "BSidesPDX_2018:C_0603" V 6815 3920 50  0001 C CNN
 F 3 "~" H 6885 3920 50  0001 C CNN
 	1    6885 3920
@@
 F 0 "R104" H 7625 3966 50  0000 L CNN
 F 1 "100R" H 7625 3875 50  0000 L CNN
-F 2 "pkl_dipol:R_0603" V 7485 3920 50  0001 C CNN
+F 2 "BSidesPDX_2018:C_0603" V 7485 3920 50  0001 C CNN
 F 3 "~" H 7555 3920 50  0001 C CNN
 	1    7555 3920
@@
 F 0 "C1" H 10205 1391 50  0000 L CNN
 F 1 "10u" H 10205 1300 50  0000 L CNN
-F 2 "pkl_dipol:C_0805" H 10128 1195 50  0001 C CNN
+F 2 "BSidesPDX_2018:C_0805" H 10128 1195 50  0001 C CNN
 F 3 "~" H 10090 1345 50  0001 C CNN
 	1    10090 1345
@@
 F 0 "C2" H 10780 1391 50  0000 L CNN
 F 1 "0.1u" H 10780 1300 50  0000 L CNN
-F 2 "pkl_dipol:C_0402" H 10703 1195 50  0001 C CNN
+F 2 "BSidesPDX_2018:C_0603" H 10703 1195 50  0001 C CNN
 F 3 "~" H 10665 1345 50  0001 C CNN
 	1    10665 1345
@@
 F 0 "R4" H 5055 1766 50  0000 L CNN
 F 1 "100R" H 5055 1675 50  0000 L CNN
-F 2 "pkl_dipol:R_0603" V 4915 1720 50  0001 C CNN
+F 2 "BSidesPDX_2018:C_0603" V 4915 1720 50  0001 C CNN
 F 3 "~" H 4985 1720 50  0001 C CNN
 	1    4985 1720
@@
 F 0 "R3" H 5955 1766 50  0000 L CNN
 F 1 "100R" H 5955 1675 50  0000 L CNN
-F 2 "pkl_dipol:R_0603" V 5815 1720 50  0001 C CNN
+F 2 "BSidesPDX_2018:C_0603" V 5815 1720 50  0001 C CNN
 F 3 "~" H 5885 1720 50  0001 C CNN
 	1    5885 1720
@@
 F 0 "R2" H 6890 1766 50  0000 L CNN
 F 1 "100R" H 6890 1675 50  0000 L CNN
-F 2 "pkl_dipol:R_0603" V 6750 1720 50  0001 C CNN
+F 2 "BSidesPDX_2018:C_0603" V 6750 1720 50  0001 C CNN
 F 3 "~" H 6820 1720 50  0001 C CNN
 	1    6820 1720
@@
 F 0 "R1" H 7790 1766 50  0000 L CNN
 F 1 "100R" H 7790 1675 50  0000 L CNN
-F 2 "pkl_dipol:R_0603" V 7650 1720 50  0001 C CNN
+F 2 "BSidesPDX_2018:C_0603" V 7650 1720 50  0001 C CNN
 F 3 "~" H 7720 1720 50  0001 C CNN
 	1    7720 1720
@@
 F 0 "S1" H 9785 4617 60  0000 C CNN
 F 1 "PTS645SM43SMTR92_LFS" H 9785 4511 60  0000 C CNN
-F 2 "digikey-footprints:Switch_Tactile_SMD_6x6mm_PTS645" H 9985 4470 60  0001 L CNN
+F 2 "BSidesPDX_2018:Switch_Tactile_SMD_6x6mm_PTS645" H 9985 4470 60  0001 L CNN
 F 3 "https://www.ckswitches.com/media/1471/pts645.pdf" H 9985 4570 60  0001 L CNN
 F 4 "CKN9112CT-ND" H 9985 4670 60  0001 L CNN "Digi-Key_PN"
@@
 F 0 "S2" H 9785 5267 60  0000 C CNN
 F 1 "PTS645SM43SMTR92_LFS" H 9785 5161 60  0000 C CNN
-F 2 "digikey-footprints:Switch_Tactile_SMD_6x6mm_PTS645" H 9985 5120 60  0001 L CNN
+F 2 "BSidesPDX_2018:Switch_Tactile_SMD_6x6mm_PTS645" H 9985 5120 60  0001 L CNN
 F 3 "https://www.ckswitches.com/media/1471/pts645.pdf" H 9985 5220 60  0001 L CNN
 F 4 "CKN9112CT-ND" H 9985 5320 60  0001 L CNN "Digi-Key_PN"
@@
 F 0 "R5" V 2490 4690 50  0000 C CNN
 F 1 "51R" V 2570 4690 50  0000 C CNN
-F 2 "pkl_dipol:R_0603" V 2500 4690 50  0001 C CNN
+F 2 "BSidesPDX_2018:C_0603" V 2500 4690 50  0001 C CNN
 F 3 "~" H 2570 4690 50  0001 C CNN
 	1    2570 4690
@@
 F 0 "R6" V 2995 4790 50  0000 C CNN
 F 1 "51R" V 3075 4790 50  0000 C CNN
-F 2 "pkl_dipol:R_0603" V 3015 4790 50  0001 C CNN
+F 2 "BSidesPDX_2018:C_0603" V 3015 4790 50  0001 C CNN
 F 3 "~" H 3085 4790 50  0001 C CNN
 	1    3085 4790
@@
 F 0 "R7" H 2910 4476 50  0000 L CNN
 F 1 "1K" H 2910 4385 50  0000 L CNN
-F 2 "pkl_dipol:R_0603" V 2770 4430 50  0001 C CNN
+F 2 "BSidesPDX_2018:C_0603" V 2770 4430 50  0001 C CNN
 F 3 "~" H 2840 4430 50  0001 C CNN
 	1    2840 4430
